File: Hardware/S80C Ver 1_0/S80C.sch (KiCad schematic (older format))
At the start: 14 parts, among them J101 02x20, J102 01x04, SW101 SW_Push, U101 Z80CPU, U102 16C550, U103 74LS14, U104 74LS04, X101 8Mhz, X102 1.8432Mhz

Commit message: Update S80C design
Parts:
- removed C101: 100pf, Capacitor_THT:C_Disc_D5.0mm_W2.5mm_P5.00mm, symbol Pynckels:C
- removed D101: 5V1, Pynckels:D_Zener_Reverse_Biased, symbol Pynckels:D_Zener
- removed J101: 02x20, Pynckels:PinSocket_2x20_P2.54mm_Vertical, symbol Connector_Generic:Conn_02x20_Odd_Even
- removed J102: 01x04, Connector_PinHeader_2.54mm:PinHeader_1x04_P2.54mm_Vertical, symbol Connector:Conn_01x04_Male
- removed U101: Z80CPU, Package_DIP:DIP-40_W15.24mm, symbol Pynckels:Z80CPU
- removed U102: 16C550, Package_DIP:DIP-40_W15.24mm, symbol Pynckels:16C550
- removed U103: 74LS14, Package_DIP:DIP-14_W7.62mm, symbol Pynckels:74LS14
- removed U104: 74LS04, Package_DIP:DIP-14_W7.62mm, symbol Pynckels:74LS04
- removed X101: 8Mhz, Oscillator:Oscillator_DIP-14, symbol Pynckels:XO32
- removed X102: 1.8432Mhz, Oscillator:Oscillator_DIP-14, symbol Pynckels:XO32
- added C101: 22µF, Capacitor_SMD:C_0603_1608Metric_Pad1.05x0.95mm_HandSolder, symbol Pynckels:C_Small
- added C103: 0.1µF, Capacitor_SMD:C_0603_1608Metric_Pad1.05x0.95mm_HandSolder, symbol Pynckels:C_Small
- added C104: 1µF, Capacitor_SMD:C_0603_1608Metric_Pad1.05x0.95mm_HandSolder, symbol Pynckels:C_Small
- added D101: SP0503BAHT, Package_TO_SOT_SMD:SOT-143, symbol Power_Protection:SP0503BAHT
- added J101: USB, digikey-kicad-library:USB_Micro_B_Female_10118192, symbol Pynckels:USB_micro
- added J102: Conn_01x14_Male, Connector_PinHeader_2.54mm:PinHeader_1x14_P2.54mm_Vertical_SMD_Pin1Left, symbol Connector:Conn_01x14_Male
- added U101: CP2105, digikey-kicad-library:QFN-24-1EP_4x4mm, symbol Pynckels:CP2105
- added U102: AS6C8008A, Package_SO:TSOP-II-44_10.16x18.41mm_P0.8mm, symbol Pynckels:AS6C8008A
- added U103: eZ80L92, digikey-kicad-library:LQFP-100_14x14mm, symbol Pynckels:eZ80L92
- added X101: SG-615PTJ 32Khz, Oscillator:Oscillator_SMD_SeikoEpson_SG8002JA-4Pin_14.0x8.7mm, symbol Oscillator:SG-615
- added X102: SG-615PTJ 50Mhz, Oscillator:Oscillator_SMD_SeikoEpson_SG8002JA-4Pin_14.0x8.7mm, symbol Oscillator:SG-615
- C102: value 22μF -> 2µF; footprint Capacitor_THT:CP_Radial_D6.3mm_P2.50mm -> Capacitor_SMD:C_0603_1608Metric_Pad1.05x0.95mm_HandSolder
- R101, R102: footprint Resistor_THT:R_Axial_DIN0207_L6.3mm_D2.5mm_P7.62mm_Horizontal -> Resistor_SMD:R_0603_1608Metric_Pad1.05x0.95mm_HandSolder
- SW101: footprint Button_Switch_THT:SW_PUSH_6mm -> Button_Switch_SMD:SW_DIP_SPSTx01_Slide_6.7x4.1mm_W8.61mm_P2.54mm_LowProfile
Connections:
- net labels added: +3V3, A16, A17, A18, A19, CTSe, CTSs, DSRe, DSRs, DTRe, DTRs, GPIO0, GPIO1, GPIO2, GPIO3, GPIO4, GPIO5, GPIO6, GPIO7, PC6, PC7, PD6, PD7, RTC_XIN, RTSe, RTSs, RxDe, RxDs, TxDe, TxDs, XIN, ~MREQ, ~RESET
- net labels removed: Address, CLKs, Control, Data, G, INT, Reset, Rx, Serial, Tx, V, ~BusAck, ~BusRq, ~CLK, ~Halt, ~INT, ~IOrq, ~M1, ~Mreq, ~NMI, ~Refresh, ~Reset, ~Wait
- wire segments 153 -> 269
- no-connect marks 11 -> 29
Other:
- note removed: "Button released: ~Reset~ = 1, T = C (R1 + R2) = 10 ms before non-active (1)\nButton pushed: ~Reset~ = 0, T = C R2 = 5 ms before active (0)\n\nRequired for Z80 @ 20Mhz: 3 clock cycles -> 150 nano sec"
- note removed: "Clipping 0V-5V"
- note removed: "External bus"
- note removed: "Later on, USB power will be clamped. For the\nmoment, an usb to ttl serial cable is used to get\npower (Vcc, Gnd) and serial communications (Rx, Tx).\n\nThe measured noise is below 100mA top-to-top and\nbelow 10mA average. So no extra bypass capacitors\nare necessary for the moment."
- note removed: "Processor"
- note removed: "Questions :\n Processor choice - Z80 or Z80182\n Memory design - Z80 + bankswitching or Z80182 with 1 Mb addressable\n Serial - 1 or 2\n Storage - Flash ?"
- note removed: "Reset - Normal & Power On"
- note removed: "Serial"
- note removed: "USB to TTL connection"
